Commit message: chore: bases

File: blazerbot_description/urdf/blazerbot_core.xacro (robot description, xacro)
@@ -4,8 +4,6 @@
 Project: Blazerbot Description (CS353 Lab 3)
 Author: Zabdiel Addo
-Email: zabdiel.addo@ashesi.edu.gh
-Version: 1.0.1
-Brief: Core robot model for Blazerbot (LIMO Agile X base): chassis + 4-wheel diff drive.
-       NOTE: LiDAR is defined in urdf/sensors/lidar.xacro as a macro.
+Version: 1.0.2
+Brief: Core robot model. base_footprint added for Nav2/AMCL/SLAM compatibility.
 -->
 <robot xmlns:xacro="http://www.ros.org/wiki/xacro">
@@ -25,7 +23,13 @@
     <xacro:property name="wheel_width" value="0.035" />
     <xacro:property name="wheel_mass" value="0.30" />
+    <!-- base_footprint: ground-plane projection, required by Nav2/AMCL/SLAM -->
+    <link name="base_footprint" />
+    <joint name="base_footprint_joint" type="fixed">
+        <parent link="base_link" />
+        <child link="base_footprint" />
+        <origin xyz="0 0 ${wheel_radius}" rpy="0 0 0" />
+    </joint>
     <!-- base_link at wheel center plane -->
     <link name="base_link" />
-    <!-- Chassis above base_link -->
     <xacro:property name="chassis_z_from_base"
         value="${ground_clearance + chassis_height/2 - wheel_radius}" />
@@ -58,5 +62,4 @@
         <material>Gazebo/Black</material>
     </gazebo>
-    <!-- Wheels attached to base_link -->
     <xacro:diff_drive_wheels
         parent_link="base_link"

File: blazerbot_description/urdf/control/gazebo_control.xacro (robot description, xacro)
@@ -9,5 +9,5 @@
        Subscribes to cmd_vel and publishes odom + tf in Gazebo for bridging to ROS 2.
 ~~~~~
-Last Modified: Tuesday, 17th February 2026 9:51:48 AM
+Last Modified: Thursday, 5th March 2026 5:28:26 PM
 Modified By: Zabdiel Addo
 ~~~~~

File: blazerbot_description/urdf/sensors/lidar.xacro (robot description, xacro)
@@ -10,6 +10,6 @@
        Publishes LaserScan data in Gazebo on the "scan" topic for wall following.
 ~~~~~
-Last Modified: Tuesday, 24th February 2026 5:26:33 PM
-Modified By: Philip Quartey
+Last Modified: Saturday, 28th February 2026 4:01:01 AM
+Modified By: Zabdiel Addo
 ~~~~~
 Copyright ©2025 Zabdiel Addo. All rights reserved.
@@ -109,5 +109,5 @@
                 <always_on>true</always_on>
                 <visualize>true</visualize>
-                <update_rate>10</update_rate>
+                <update_rate>20</update_rate>
                 <lidar>
                     <scan>
